Commit message: dolly navigation added

File: dolly_description/urdf/dolly.urdf (robot description, URDF)
Before this commit: robot Dolly, 6 links, 5 joints
Links:
- removed link chassis
- added link base_footprint
- added link base_link, mass 1.0; visual box size=1.0 0.5 0.15; visual box size=1.0 0.5 0.15
Joints:
- added joint base_joint: type fixed, parent base_footprint, child base_link, origin xyz=0.0 0.0 0.010 rpy=0 0 0
- joint caster_front_wheel: parent chassis -> base_link
- joint caster_wheel: parent chassis -> base_link
- joint left_wheel_joint: parent chassis -> base_link
- joint right_wheel_joint: parent chassis -> base_link
- joint scan_joint: parent chassis -> base_link
